File: PCB/PaperDox.kicad_pcb (KiCad board)
At the start: 2 copper layers, 80 parts, among them U1 nice_nano

Commit message: some wip
Parts:
- moved U1 3.88 mm to (157.3, 38.6)
Routing:
- net Net-(D36-A): track 0.00 -> 161.8 mm
- net Net-(D35-A): track 0.00 -> 141.5 mm
- net Net-(D34-A): track 0.00 -> 130.0 mm
- net Net-(D30-A): track 0.00 -> 127.9 mm
- net Net-(D33-A): track 0.00 -> 120.2 mm
- net Net-(D25-A): track 0.00 -> 114.6 mm
- net Net-(D20-A): track 0.00 -> 111.1 mm
- net /COL0: track 0.83 -> 110.6 mm
- net Net-(D10-A): track 0.00 -> 105.1 mm
- net /COL1: track 0.00 -> 101.8 mm
- net Net-(D29-A): track 0.00 -> 98.7 mm
- net /COL2: track 0.00 -> 94.8 mm
- net Net-(D24-A): track 0.00 -> 93.2 mm
- net Net-(D5-A): track 0.00 -> 89.2 mm
- net Net-(D15-A): track 0.00 -> 88.6 mm
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