File: PCB/PaperDox.kicad_sch (KiCad schematic)
At the start: 44 parts, among them SW0:10 SW0:3, SW0:11 SW0:2, SW0:12 SW0:1, SW0:7 SW0:6, SW0:8 SW0:5, SW0:9 SW0:4, SW1:10 SW1:3, SW1:11 SW1:2, SW1:12 SW1:1, SW1:13 SW1:0, SW1:9 SW1:4, SW2:10 SW2:3, SW2:11 SW2:2, SW2:12 SW2:1, SW2:13 SW2:0, SW2:7 SW2:6, SW2:8 SW2:5, SW2:9 SW2:4, SW3:10 SW3:3, SW3:11 SW3:2, SW3:12 SW3:1, SW3:13 SW3:0, SW3:8 SW3:5, SW3:9 SW3:4, SW4:10 SW4:3, SW4:11 SW4:2, SW4:12 SW4:1, SW4:13 SW4:0, SW4:7 SW4:6, SW4:8 SW4:5, SW4:9 SW4:4, SW5:10 SW5:3, SW5:11 SW5:2, SW5:12 SW5:1, SW5:13 SW5:0, SW5:7 SW5:6, SW5:8 SW5:5, SW5:9 SW5:4

Commit message: i should commit and push this huh
Parts:
- removed D1:7, D1:8: D, symbol ErgoDOX-rescue:DIODE
- removed SW0:10: SW0:3, symbol ErgoDOX-rescue:SWITCH_DIODE
- removed SW0:11: SW0:2, symbol ErgoDOX-rescue:SWITCH_DIODE
- removed SW0:12: SW0:1, symbol ErgoDOX-rescue:SWITCH_DIODE
- removed SW0:7: SW0:6, symbol ErgoDOX-rescue:SWITCH_DIODE
- removed SW0:8: SW0:5, symbol ErgoDOX-rescue:SWITCH_DIODE
- removed SW0:9: SW0:4, symbol ErgoDOX-rescue:SWITCH_DIODE
- removed SW1:10: SW1:3, symbol ErgoDOX-rescue:SWITCH_DIODE
- removed SW1:11: SW1:2, symbol ErgoDOX-rescue:SWITCH_DIODE
- removed SW1:12: SW1:1, symbol ErgoDOX-rescue:SWITCH_DIODE
- removed SW1:13: SW1:0, symbol ErgoDOX-rescue:SWITCH_DIODE
- removed SW1:9: SW1:4, symbol ErgoDOX-rescue:SWITCH_DIODE
- removed SW2:10: SW2:3, symbol ErgoDOX-rescue:SWITCH_DIODE
- removed SW2:11: SW2:2, symbol ErgoDOX-rescue:SWITCH_DIODE
- removed SW2:12: SW2:1, symbol ErgoDOX-rescue:SWITCH_DIODE
- removed SW2:13: SW2:0, symbol ErgoDOX-rescue:SWITCH_DIODE
- removed SW2:7: SW2:6, symbol ErgoDOX-rescue:SWITCH_DIODE
- removed SW2:8: SW2:5, symbol ErgoDOX-rescue:SWITCH_DIODE
- removed SW2:9: SW2:4, symbol ErgoDOX-rescue:SWITCH_DIODE
- removed SW3:10: SW3:3, symbol ErgoDOX-rescue:SWITCH_DIODE
- removed SW3:11: SW3:2, symbol ErgoDOX-rescue:SWITCH_DIODE
- removed SW3:12: SW3:1, symbol ErgoDOX-rescue:SWITCH_DIODE
- removed SW3:13: SW3:0, symbol ErgoDOX-rescue:SWITCH_DIODE
- removed SW3:8: SW3:5, symbol ErgoDOX-rescue:SWITCH_DIODE
- removed SW3:9: SW3:4, symbol ErgoDOX-rescue:SWITCH_DIODE
- removed SW4:10: SW4:3, symbol ErgoDOX-rescue:SWITCH_DIODE
- removed SW4:11: SW4:2, symbol ErgoDOX-rescue:SWITCH_DIODE
- removed SW4:12: SW4:1, symbol ErgoDOX-rescue:SWITCH_DIODE
- removed SW4:13: SW4:0, symbol ErgoDOX-rescue:SWITCH_DIODE
- removed SW4:7: SW4:6, symbol ErgoDOX-rescue:SWITCH_DIODE
- removed SW4:8: SW4:5, symbol ErgoDOX-rescue:SWITCH_DIODE
- removed SW4:9: SW4:4, symbol ErgoDOX-rescue:SWITCH_DIODE
- removed SW5:10: SW5:3, symbol ErgoDOX-rescue:SWITCH_DIODE
- removed SW5:11: SW5:2, symbol ErgoDOX-rescue:SWITCH_DIODE
- removed SW5:12: SW5:1, symbol ErgoDOX-rescue:SWITCH_DIODE
- removed SW5:13: SW5:0, symbol ErgoDOX-rescue:SWITCH_DIODE
- removed SW5:7: SW5:6, symbol ErgoDOX-rescue:SWITCH_DIODE
- removed SW5:8: SW5:5, symbol ErgoDOX-rescue:SWITCH_DIODE
- removed SW5:9: SW5:4, symbol ErgoDOX-rescue:SWITCH_DIODE
- removed SX0:10: SX0:3, symbol ErgoDOX-rescue:SWITCH_PUSH
- removed SX0:11: SX0:2, symbol ErgoDOX-rescue:SWITCH_PUSH
- removed SX1:7: SX1:6, symbol ErgoDOX-rescue:SWITCH_PUSH
- removed SX1:8: SX1:5, symbol ErgoDOX-rescue:SWITCH_PUSH
- added D1, D10, D11, D12, D13, D14, D15, D16, D17, D18, D19, D2, D20, D21, D22, D23, D24, D25, D26, D27, D28, D29, D3, D30, D31, D32, D33, D34, D35, D36, D38, D39, D4, D5, D6, D7, D8, D9: 1N4148, keyboard_reversible:ComboDiode, symbol Diode:1N4148
- added KSW1, KSW10, KSW11, KSW12, KSW13, KSW14, KSW15, KSW16, KSW17, KSW18, KSW19, KSW2, KSW20, KSW22, KSW23, KSW24, KSW25, KSW26, KSW27, KSW28, KSW29, KSW3, KSW30, KSW31, KSW32, KSW33, KSW34, KSW35, KSW36, KSW37, KSW38, KSW39, KSW4, KSW5, KSW6, KSW7, KSW8, KSW9: Keyswitch, keyboard_reversible:Choc_Hotswap, symbol Switch:SW_Push
- added RST1: SW_Push, Button_Switch_THT:SW_PUSH_6mm, symbol Switch:SW_Push
- added U1: nice_nano, keyboard_reversible:ProMicro_Mill-Max, symbol nice_nano:nice_nano
Connections:
- net COL0: now also D1.1 (K), D2.1 (K), D3.1 (K), D4.1 (K), D5.1 (K), U1.13 (NFC1/P0.09)
- net COL1: now also D10.1 (K), D6.1 (K), D7.1 (K), D8.1 (K), D9.1 (K), U1.14 (NFC2/P0.10)
- net COL4: now also D21.1 (K), D22.1 (K), D23.1 (K), D24.1 (K), D25.1 (K), U1.17 (P1.15)
- net COL5: now also D26.1 (K), D27.1 (K), D28.1 (K), D29.1 (K), D30.1 (K), U1.18 (AIN0/P0.02)
- net COL6: now also D31.1 (K), D32.1 (K), D33.1 (K), U1.19 (AIN5/P0.29)
- net ROW0: now also KSW35.2, KSW36.2, KSW37.2, KSW38.2, KSW39.2, U1.12 (P1.06)
- net ROW1: now also KSW29.2, KSW30.2, KSW31.2, KSW32.2, KSW33.2, KSW34.2, U1.11 (P1.04)
- net ROW2: now also KSW22.2, KSW23.2, KSW24.2, KSW25.2, KSW26.2, KSW27.2, U1.10 (P0.11)
- net ROW3: now also KSW15.2, KSW16.2, KSW17.2, KSW18.2, KSW19.2, KSW20.2, KSW28.2, U1.9 (P1.00)
- net ROW4: now also KSW10.2, KSW11.2, KSW12.2, KSW13.2, KSW14.2, KSW8.2, KSW9.2, U1.8 (P0.24)
- net ROW5: now also KSW1.2, KSW2.2, KSW3.2, KSW4.2, KSW5.2, KSW6.2, KSW7.2, U1.7 (P0.22)
- new net: D3.2 (A), KSW15.1
- new net: D36.2 (A), KSW37.1
- new net: D23.2 (A), KSW19.1
- new net: D12.2 (A), KSW10.1
- new net: D17.2 (A), KSW11.1
- new net: D32.2 (A), KSW14.1
- new net: D29.2 (A), KSW27.1
- new net: D35.2 (A), KSW38.1
- new net: D8.2 (A), KSW16.1
- new net: D31.2 (A), KSW7.1
- new net: D27.2 (A), KSW13.1
- new net: D15.2 (A), KSW31.1
- new net: D33.2 (A), KSW28.1
- new net: D26.2 (A), KSW6.1
- new net: D11.2 (A), KSW3.1
- new net: D20.2 (A), KSW32.1
- new net: D38.2 (A), KSW36.1
- new net: D13.2 (A), KSW17.1
- new net: D22.2 (A), KSW12.1
- new net: D34.2 (A), KSW39.1
- new net: D6.2 (A), KSW2.1
- new net: D24.2 (A), KSW26.1
- new net: D14.2 (A), KSW24.1
- new net: D18.2 (A), KSW18.1
- new net: D16.2 (A), KSW4.1
- new net: D19.2 (A), KSW25.1
- new net: D1.2 (A), KSW1.1
- new net: D9.2 (A), KSW23.1
- new net: D7.2 (A), KSW9.1
- new net: D10.2 (A), KSW30.1
- new net: D21.2 (A), KSW5.1
- new net: D4.2 (A), KSW22.1
- new net: RST1.1, U1.23 (GND)
- new net: RST1.2, U1.22 (RST)
- new net: D25.2 (A), KSW33.1
- new net: D28.2 (A), KSW20.1
- new net: D30.2 (A), KSW34.1
- new net: D5.2 (A), KSW29.1
- new net: D2.2 (A), KSW8.1
- new net: D39.2 (A), KSW35.1
- new net COL2: D11.1 (K), D12.1 (K), D13.1 (K), D14.1 (K), D15.1 (K), U1.15 (P1.11)
- new net COL3: D16.1 (K), D17.1 (K), D18.1 (K), D19.1 (K), D20.1 (K), U1.16 (P1.13)
- new net COL7: D34.1 (K), D35.1 (K), D36.1 (K), D38.1 (K), D39.1 (K), U1.20 (AIN7/P0.31)
Other:
- company: (none) -> TheHonker
- title: (none) -> PaperDox

Commit message: some wip
Parts:
- renumbered D38 to D37, D39 to D38, RST1 to RST
Changed lines of the file:
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@@
 	(wire
 		(pts
-			(xy 166.37 119.38) (xy 147.32 119.38)
-		)
-		(stroke
-			(width 0)
-			(type default)
-		)
-	)
-	(wire
-		(pts
 			(xy 125.73 46.99) (xy 128.27 46.99)
 		)
@@
 	(wire
 		(pts
-			(xy 166.37 53.34) (xy 166.37 119.38)
-		)
-		(stroke
-			(width 0)
-			(type default)
-		)
-	)
-	(wire
-		(pts
 			(xy 128.27 59.69) (xy 118.11 59.69)
 		)
@@
 	(wire
 		(pts
+			(xy 147.32 124.46) (xy 166.37 124.46)
+		)
+		(stroke
+			(width 0)
+			(type default)
+		)
+	)
+	(wire
+		(pts
 			(xy 71.12 46.99) (xy 71.12 48.26)
 		)
@@
 	(wire
 		(pts
-			(xy 147.32 119.38) (xy 147.32 151.13)
+			(xy 147.32 124.46) (xy 147.32 151.13)
 		)
 		(stroke
@@
 	(wire
 		(pts
+			(xy 166.37 53.34) (xy 166.37 124.46)
+		)
+		(stroke
+			(width 0)
+			(type default)
+		)
+	)
+	(wire
+		(pts
 			(xy 115.57 107.95) (xy 119.38 107.95)
 		)
@@
 		(dnp no)
 		(fields_autoplaced yes)
-		(property "Reference" "D38"
+		(property "Reference" "D37"
 			(at 168.91 49.5299 90)
 			(effects
@@
 			(project "PaperDox"
 				(path "/401f1071-09ae-4313-b595-796f076eb7fc"
-					(reference "D38")
+					(reference "D37")
 					(unit 1)
 				)
@@
 		(on_board yes)
 		(dnp no)
-		(fields_autoplaced yes)
-		(property "Reference" "RST1"
-			(at 251.46 44.958 0)
+		(property "Reference" "RST"
+			(at 251.46 45.212 0)
 			(effects
 				(font
@@
 			(project ""
 				(path "/401f1071-09ae-4313-b595-796f076eb7fc"
-					(reference "RST1")
+					(reference "RST")
 					(unit 1)
 				)
@@
 		(dnp no)
 		(fields_autoplaced yes)
-		(property "Reference" "D39"
-			(at 161.29 48.2599 90)
+		(property "Reference" "D38"
+			(at 166.37 48.2599 90)
 			(effects
 				(font
 					(size 1.27 1.27)
 				)
-				(justify right)
+				(justify left)
 			)
 		)
@@
 			(project "PaperDox"
 				(path "/401f1071-09ae-4313-b595-796f076eb7fc"
-					(reference "D39")
+					(reference "D38")
 					(unit 1)
 				)
